File: pcb/relay_controller.kicad_pcb (KiCad board)
At the start: 2 copper layers, 118.1 x 55.1 mm, 58 parts, among them P1 PWR_JACK_2.5x5.5, P10 HEADER_02X08_SMD, P11 HEADER_02X08_SMD, P2 HEADER_01X03_SMD_RA, P3 HEADER_01X03_SMD_RA, P4 HEADER_01X03_SMD_RA, P5 HEADER_01X03_SMD_RA, P6 HEADER_01X02_SMD_RA, P7 BNC_DOUBLE_RA, P8 HEADER_02X08_SMD, P9 HEADER_02X08_SMD, SW1 SPST_SLIDE_AS, U1 TLE7230R, U2 TLE7230R, U3 TLE7230R, U4 TLE7230R

Commit message: More progress towards pcb1.0.
Parts:
- removed C4, C5, C6, C7: 0.1uF, relay_controller:SM1210
- removed D1, D10, D11, D12, D13, D14, D15, D16, D17, D18, D19, D2, D20, D21, D22, D23, D24, D25, D26, D27, D28, D29, D3, D30, D31, D32, D33, D4, D5, D6, D7, D8, D9: LED_24V, relay_controller:LED_555-3XXX
- removed P10, P11, P8, P9: HEADER_02X08_SMD, relay_controller:HEADER_02x08_SMD
- added L1: LED_24V, relay_controller:LED_555-3XXX, F.Cu at (201.9, 94.0)
- added L2: LED_5V_GRN, relay_controller:LED_555-3XXX, F.Cu at (120.0, 101.6)
- added L3: LED_5V_GRN, relay_controller:LED_555-3XXX, F.Cu at (140.3, 101.6)
- added L4: LED_5V_GRN, relay_controller:LED_555-3XXX, F.Cu at (160.7, 101.6)
- added L5: LED_5V_GRN, relay_controller:LED_555-3XXX, F.Cu at (181.0, 101.6)
- added L6: LED_5V_GRN, relay_controller:LED_555-3XXX, F.Cu at (120.0, 123.2)
- added L7: LED_5V_GRN, relay_controller:LED_555-3XXX, F.Cu at (140.3, 123.2)
- added L8: LED_5V_GRN, relay_controller:LED_555-3XXX, F.Cu at (160.7, 123.2)
- added L9: LED_5V_GRN, relay_controller:LED_555-3XXX, F.Cu at (181.0, 123.2)
- added R1: 5.11k, relay_controller:SM1210, B.Cu at (201.3, 90.8)
- added R10: 150, relay_controller:SM1210, B.Cu at (181.0, 120.7)
- added R2: 1k, relay_controller:SM1210, B.Cu at (201.3, 97.2)
- added R3: 150, relay_controller:SM1210, B.Cu at (120.0, 99.1)
- added R4: 150, relay_controller:SM1210, B.Cu at (140.3, 99.1)
- added R5: 150, relay_controller:SM1210, B.Cu at (160.7, 99.1)
- added R6: 150, relay_controller:SM1210, B.Cu at (181.0, 99.1)
- added R7: 150, relay_controller:SM1210, B.Cu at (120.0, 120.7)
- added R8: 150, relay_controller:SM1210, B.Cu at (140.3, 120.7)
- added R9: 150, relay_controller:SM1210, B.Cu at (160.7, 120.7)
- added T1: TERM_BLK_ANG_2_PIN, relay_controller:TERM_BLK_ANG_2_PIN, F.Cu at (120.0, 94.6)
- added T2: TERM_BLK_ANG_2_PIN, relay_controller:TERM_BLK_ANG_2_PIN, F.Cu at (140.3, 94.6)
- added T3: TERM_BLK_ANG_2_PIN, relay_controller:TERM_BLK_ANG_2_PIN, F.Cu at (160.7, 94.6)
- added T4: TERM_BLK_ANG_2_PIN, relay_controller:TERM_BLK_ANG_2_PIN, F.Cu at (181.0, 94.6)
- added T5: TERM_BLK_ANG_2_PIN, relay_controller:TERM_BLK_ANG_2_PIN, F.Cu at (120.0, 116.2)
- added T6: TERM_BLK_ANG_2_PIN, relay_controller:TERM_BLK_ANG_2_PIN, F.Cu at (140.3, 116.2)
- added T7: TERM_BLK_ANG_2_PIN, relay_controller:TERM_BLK_ANG_2_PIN, F.Cu at (160.7, 116.2)
- added T8: TERM_BLK_ANG_2_PIN, relay_controller:TERM_BLK_ANG_2_PIN, F.Cu at (181.0, 116.2)
- added U5: SSR_DC_6PIN, relay_controller:ASSR-1611, B.Cu at (120.0, 108.6)
- added U6: SSR_DC_6PIN, relay_controller:ASSR-1611, B.Cu at (140.3, 108.6)
- added U7: SSR_DC_6PIN, relay_controller:ASSR-1611, B.Cu at (160.7, 108.6)
- added U8: SSR_DC_6PIN, relay_controller:ASSR-1611, B.Cu at (181.0, 108.6)
- U1, U2, U3, U4: value TLE7230R -> SSR_DC_6PIN; footprint relay_controller:PG-DSO-36 -> relay_controller:ASSR-1611
- moved U1 60.4 mm to (120.0, 87.0)
- moved U4 43.9 mm to (181.0, 87.0)
- moved U3 31.6 mm to (160.7, 87.0)
- moved U2 4.84 mm to (140.3, 87.0)
Connections:
- ARDUINO1 pad 22: (no net) -> /LED_0
- ARDUINO1 pad 23: (no net) -> /LED_1
- ARDUINO1 pad 24: (no net) -> /LED_2
- ARDUINO1 pad 25: (no net) -> /LED_3
- ARDUINO1 pad 26: (no net) -> /LED_4
- ARDUINO1 pad 27: (no net) -> /LED_5
- ARDUINO1 pad 28: (no net) -> /LED_6
- ARDUINO1 pad 29: (no net) -> /LED_7
- ARDUINO1 pad 33: (no net) -> /LED_PWR_IN
- ARDUINO1 pad 38: (no net) -> /RELAY_0
- ARDUINO1 pad 39: (no net) -> /RELAY_1
- ARDUINO1 pad 40: (no net) -> /RELAY_2
- ARDUINO1 pad 41: (no net) -> /RELAY_3
- ARDUINO1 pad 42: (no net) -> /RELAY_4
- ARDUINO1 pad 43: (no net) -> /RELAY_5
- ARDUINO1 pad 44: /RESET -> /RELAY_6
- ARDUINO1 pad 45: (no net) -> /RELAY_7
- ARDUINO1 pad 46: /CS -> (no net)
- ARDUINO1 pad 50: /MISO -> (no net)
- ARDUINO1 pad 51: /MOSI -> (no net)
- ARDUINO1 pad 52: /SCK -> (no net)
- ARDUINO1 pad 5V_1: +5V -> (no net)
- U1 pad 1: GND -> Net-(R3-Pad1)
- U1 pad 2: (no net) -> GND
- U1 pad 4: /OUT0 -> /OUT_0+
- U1 pad 5: /OUT1 -> /OUT_0-
- U1 pad 6: GND -> /OUT_0+
- U2 pad 1: GND -> Net-(R4-Pad1)
- U2 pad 2: (no net) -> GND
- U2 pad 4: /OUT8 -> /OUT_1+
- U2 pad 5: /OUT9 -> /OUT_1-
- U2 pad 6: GND -> /OUT_1+
- U3 pad 1: GND -> Net-(R5-Pad1)
- U3 pad 2: (no net) -> GND
- U3 pad 4: /OUT16 -> /OUT_2+
- U3 pad 5: /OUT17 -> /OUT_2-
- U3 pad 6: GND -> /OUT_2+
- U4 pad 1: GND -> Net-(R6-Pad1)
- U4 pad 2: (no net) -> GND
- U4 pad 4: /OUT24 -> /OUT_3+
- U4 pad 5: /OUT25 -> /OUT_3-
- U4 pad 6: GND -> /OUT_3+
Routing:
- net GND: track 558.3 -> 0.00 mm, vias 1 -> 0
- net VAA: track 217.8 -> 0.00 mm, vias 1 -> 0
- net +5V: track 216.2 -> 0.00 mm, vias 4 -> 0
- net /LED_PWR: track 207.8 -> 0.00 mm, vias 1 -> 0
- net /SCK: track 112.7 -> 0.00 mm, vias 5 -> 0
- net /RESET: track 97.9 -> 0.00 mm, vias 1 -> 0
- net /CS: track 96.8 -> 0.00 mm, vias 2 -> 0
- net /BNC_A: track 91.3 -> 0.00 mm
- net /TX3: track 85.3 -> 0.00 mm
- net /RX0: track 70.0 -> 0.00 mm
- net /RX3: track 65.1 -> 0.00 mm, vias 1 -> 0
- net /MISO: track 62.2 -> 0.00 mm, vias 1 -> 0
- net /SO2: track 61.2 -> 0.00 mm
- net /TX0: track 58.4 -> 0.00 mm
- net /BNC_B: track 56.7 -> 0.00 mm
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- removed copper zone on B.Cu, net GND
- removed copper zone on F.Cu, net VAA
Other:
- board text added: "Janelia Modular Device relay_controller model_number: 1190 04/2016 ver 1.0"
- board text removed: "10"
- board text removed: "11"
- board text removed: "12"
- board text removed: "13"
- board text removed: "14"
- board text removed: "15"
- board text removed: "16"
- board text removed: "17"
- board text removed: "18"
- board text removed: "19"
- board text removed: "20"
- board text removed: "21"
- board text removed: "22"
- board text removed: "23"
- board text removed: "24"
- board text removed: "25"
- board text removed: "26"
- board text removed: "27"
- board text removed: "28"
- board text removed: "29"
- board text removed: "30"
- board text removed: "31"
- board text removed: "8"
- board text removed: "9"
- board text removed: "Janelia Modular Device relay_controller model_number: 1110 03/2016 ver 1.5"

Commit message: pcb1.0 completed.
Parts:
- turned U6 to 270 degrees
Routing:
- net GND: track 0.00 -> 410.8 mm
- net VAA: track 0.00 -> 149.0 mm
- net /LED_4: track 0.00 -> 92.4 mm, vias 0 -> 1
- net /BNC_A: track 0.00 -> 91.3 mm
- net /TX3: track 0.00 -> 85.2 mm
- net /LED_5: track 0.00 -> 83.6 mm, vias 0 -> 1
- net /LED_0: track 0.00 -> 83.4 mm
- net /RELAY_4: track 0.00 -> 76.1 mm, vias 0 -> 1
- net /RELAY_0: track 0.00 -> 76.1 mm, vias 0 -> 1
- net /RX3: track 0.00 -> 71.2 mm, vias 0 -> 1
- net /RX0: track 0.00 -> 70.0 mm
- net /BNC_B: track 0.00 -> 65.7 mm
- net /LED_1: track 0.00 -> 65.0 mm
- net /RELAY_1: track 0.00 -> 63.4 mm, vias 0 -> 1
- net /RELAY_5: track 0.00 -> 63.1 mm, vias 0 -> 1
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- added copper zone on B.Cu, net GND
- added copper zone on F.Cu, net GND

Commit message: Switched LED_PWR to LED_GND.
Parts:
- removed R10, R9: 150, relay_controller:SM1210
- R1: value 5.11k -> 487
- R2: value 1k -> 487
- R3, R4, R5, R6, R7, R8: value 150 -> 487
- moved R1 81.7 mm to (120.0, 99.1), turned to 0 degrees
- moved R2 61.0 mm to (140.3, 99.1)
- moved R5 46.0 mm to (120.0, 120.7)
- moved R6 46.0 mm to (140.3, 120.7)
- moved R3 40.6 mm to (160.7, 99.1)
- moved R7 40.6 mm to (160.7, 120.7)
- moved R4 40.6 mm to (181.0, 99.1)
- moved R8 40.6 mm to (181.0, 120.7)
- turned L1 to 90 degrees
- turned L2 to 270 degrees
- turned L3 to 270 degrees
- turned L4 to 270 degrees
- turned L5 to 270 degrees
- turned L6 to 270 degrees
- turned L7 to 270 degrees
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Connections:
- ARDUINO1 pad 22: /LED_0 -> (no net)
- ARDUINO1 pad 23: /LED_1 -> (no net)
- ARDUINO1 pad 24: /LED_2 -> (no net)
- ARDUINO1 pad 25: /LED_3 -> (no net)
- ARDUINO1 pad 26: /LED_4 -> (no net)
- ARDUINO1 pad 27: /LED_5 -> (no net)
- ARDUINO1 pad 28: /LED_6 -> (no net)
- ARDUINO1 pad 29: /LED_7 -> (no net)
- ARDUINO1 pad 33: /LED_PWR_IN -> (no net)
- L1 pad 1: /LED_PWR -> VAA
- L1 pad 2: GND -> /LED_GND
- L2 pad 1: /LED_0 -> /RELAY_0
- L2 pad 2: GND -> /LED_GND
- L3 pad 1: /LED_1 -> /RELAY_1
- L3 pad 2: GND -> /LED_GND
- L4 pad 1: /LED_2 -> /RELAY_2
- L4 pad 2: GND -> /LED_GND
- L5 pad 1: /LED_3 -> /RELAY_3
- L5 pad 2: GND -> /LED_GND
- L6 pad 1: /LED_4 -> /RELAY_4
- L6 pad 2: GND -> /LED_GND
- L7 pad 1: /LED_5 -> /RELAY_5
- L7 pad 2: GND -> /LED_GND
- L8 pad 1: /LED_6 -> /RELAY_6
- L8 pad 2: GND -> /LED_GND
- L9 pad 1: /LED_7 -> /RELAY_7
- L9 pad 2: GND -> /LED_GND
- R1 pad 1: /LED_PWR -> Net-(R1-Pad1)
- R1 pad 2: /LED_PWR_IN -> /RELAY_0
- R2 pad 1: /LED_PWR_IN -> Net-(R2-Pad1)
- R2 pad 2: GND -> /RELAY_1
- R3 pad 2: /RELAY_0 -> /RELAY_2
- R4 pad 2: /RELAY_1 -> /RELAY_3
- R5 pad 2: /RELAY_2 -> /RELAY_4
- R6 pad 2: /RELAY_3 -> /RELAY_5
- R7 pad 2: /RELAY_4 -> /RELAY_6
- R8 pad 2: /RELAY_5 -> /RELAY_7
- SW1 pad 1: VAA -> GND
- SW1 pad 3: /LED_PWR -> /LED_GND
- U1 pad 1: Net-(R3-Pad1) -> Net-(R1-Pad1)
- U2 pad 1: Net-(R4-Pad1) -> Net-(R2-Pad1)
- U3 pad 1: Net-(R5-Pad1) -> Net-(R3-Pad1)
- U4 pad 1: Net-(R6-Pad1) -> Net-(R4-Pad1)
- U5 pad 1: Net-(R7-Pad1) -> Net-(R5-Pad1)
- U6 pad 1: Net-(R8-Pad1) -> Net-(R6-Pad1)
- U7 pad 1: Net-(R9-Pad1) -> Net-(R7-Pad1)
- U8 pad 1: Net-(R10-Pad1) -> Net-(R8-Pad1)
Routing:
- net /LED_GND: track 0.00 -> 214.0 mm
- net /LED_4: track 92.4 -> 0.00 mm, vias 1 -> 0
- net /LED_5: track 83.6 -> 0.00 mm, vias 1 -> 0
- net /LED_0: track 83.4 -> 0.00 mm
- net /LED_1: track 65.0 -> 0.00 mm
- net GND: track 410.8 -> 355.2 mm
- net /LED_7: track 54.5 -> 0.00 mm
- net /LED_6: track 51.8 -> 0.00 mm
- net /LED_2: track 41.0 -> 0.00 mm
- net /LED_PWR: track 29.9 -> 0.00 mm
- net /LED_3: track 27.7 -> 0.00 mm
- net Net-(R1-Pad1): track 0.00 -> 18.9 mm
- net Net-(R2-Pad1): track 0.00 -> 18.9 mm
- net Net-(R9-Pad1): track 18.9 -> 0.00 mm
- net Net-(R10-Pad1): track 18.9 -> 0.00 mm
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Other:
- board text added: "Janelia Modular Device relay_controller model_number: 1190 04/2016 ver 1.1"
- board text removed: "Janelia Modular Device relay_controller model_number: 1190 04/2016 ver 1.0"

Commit message: Made changes to 1.1, must complete before manufacturing boards.
Parts:
- R1, R2, R3, R4, R5, R6, R7, R8: value 487 -> 249
Connections:
- ARDUINO1 pad 10: (no net) -> /RELAY_2
- ARDUINO1 pad 11: (no net) -> /RELAY_3
- ARDUINO1 pad 12: (no net) -> /RELAY_4
- ARDUINO1 pad 38: /RELAY_0 -> (no net)
- ARDUINO1 pad 39: /RELAY_1 -> (no net)
- ARDUINO1 pad 40: /RELAY_2 -> (no net)
- ARDUINO1 pad 41: /RELAY_3 -> (no net)
- ARDUINO1 pad 42: /RELAY_4 -> (no net)
- ARDUINO1 pad 43: /RELAY_5 -> (no net)
- ARDUINO1 pad 44: /RELAY_6 -> /RELAY_5
- ARDUINO1 pad 45: /RELAY_7 -> /RELAY_6
- ARDUINO1 pad 46: (no net) -> /RELAY_7
- ARDUINO1 pad 8: (no net) -> /RELAY_0
- ARDUINO1 pad 9: (no net) -> /RELAY_1
Routing:
- net /RELAY_3: track 15.7 -> 68.9 mm
- net /RELAY_0: track 75.1 -> 35.7 mm
- net /RELAY_4: track 81.1 -> 52.6 mm
- net /RELAY_1: track 57.9 -> 30.1 mm
- net /RELAY_2: track 34.7 -> 55.9 mm
- net GND: track 355.2 -> 375.8 mm
- net VAA: track 156.9 -> 140.5 mm
- net /BNC_A: track 105.7 -> 91.5 mm
- net /RX3: track 62.7 -> 74.7 mm
- net /RELAY_5: track 62.5 -> 57.2 mm, vias 0 -> 1
- net /LED_GND: track 214.0 -> 209.7 mm
- net /RELAY_7: track 21.2 -> 17.3 mm
- net /BNC_B: track 64.8 -> 67.9 mm
- net /TX3: track 84.9 -> 83.4 mm
- net /RELAY_6: track 38.5 -> 39.5 mm, vias 0 -> 1
- removed copper zone on B.Cu, net GND
- removed copper zone on F.Cu, net GND

Commit message: Removed traces.
Routing:
- net GND: track 375.8 -> 0.00 mm
- net /LED_GND: track 209.7 -> 0.00 mm
- net VAA: track 140.5 -> 0.00 mm
- net /BNC_A: track 91.5 -> 0.00 mm
- net /TX3: track 83.4 -> 0.00 mm
- net /RX3: track 74.7 -> 0.00 mm
- net /RX0: track 70.0 -> 0.00 mm
- net /RELAY_3: track 68.9 -> 0.00 mm
- net /BNC_B: track 67.9 -> 0.00 mm
- net /TX0: track 58.4 -> 0.00 mm
- net /RELAY_5: track 57.2 -> 0.00 mm, vias 1 -> 0
- net /RELAY_2: track 55.9 -> 0.00 mm
- net /V_IN: track 54.7 -> 0.00 mm
- net /RELAY_4: track 52.6 -> 0.00 mm
- net /RX1: track 39.5 -> 0.00 mm
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